File: Hardware/spider-robot-controller.sch (KiCad schematic (older format))
At the start: 24 parts, among them CON1 AVR-ISP-6, IC1 ATMEGA328-P, P1 SERVO_HEADER, P10 SERVO_HEADER, P11 SERVO_HEADER, P12 SERVO_HEADER, P2 SERVO_HEADER, P3 SERVO_HEADER, P4 SERVO_HEADER, P5 SERVO_HEADER, P6 SERVO_HEADER, P7 SERVO_HEADER, P8 SERVO_HEADER, P9 SERVO_HEADER, SW1 SW_PUSH, Y1 16MHz

Commit message: finished schematics
Parts:
- added R2: 330, Resistors_ThroughHole:Resistor_Horizontal_RM10mm, symbol R
- added R3: 660, Resistors_ThroughHole:Resistor_Horizontal_RM10mm, symbol R
- C1, C2: footprint (none) -> Capacitors_ThroughHole:C_Disc_D3_P2.5
- C3: renamed from C?; footprint (none) -> Capacitors_ThroughHole:C_Radial_D10_L13_P5
- C4: renamed from C?; footprint (none) -> Capacitors_ThroughHole:C_Radial_D5_L6_P2.5
- CON2: renamed from CON?; footprint (none) -> library:BARREL_JACK
- P1, P10, P11, P12, P2, P3, P4, P5, P6, P7, P8, P9: footprint (none) -> Pin_Headers:Pin_Header_Angled_1x03
- P13: renamed from P?; footprint (none) -> Pin_Headers:Pin_Header_Angled_1x06
- R1: footprint (none) -> Resistors_ThroughHole:Resistor_Horizontal_RM10mm
- U1: renamed from U?; footprint (none) -> library:LM7805
- Y1: footprint (none) -> Crystals:Crystal_HC49-U_Vertical
Connections:
- net BRX: now also R2.1; no longer P13.2 (P2)
- net GND: now also R3.2
- new net: P13.2 (P2), R2.2, R3.1
Other:
- note added: "BLUETOOTH CIRCUIT"
- note added: "POWER CIRCUIT"
- moved on the sheet: P13, R1, SW1
Changed lines of the file:
@@
 Text GLabel 9200 1550 2    60   Input ~ 0
 SCK
-Text GLabel 9950 2850 0    60   Input ~ 0
-VCC
-Text GLabel 10200 2750 0    60   Input ~ 0
+Text GLabel 7050 5800 0    60   Input ~ 0
+VCC
+Text GLabel 7300 5700 0    60   Input ~ 0
 GND
 Text GLabel 6750 3250 0    60   Input ~ 0
@@
 L SW_PUSH SW1
 U 1 1 55F95F04
-P 9550 4050
-F 0 "SW1" H 9700 4160 50  0000 C CNN
-F 1 "SW_PUSH" H 9550 3970 50  0000 C CNN
-F 2 "" H 9550 4050 60  0000 C CNN
-F 3 "" H 9550 4050 60  0000 C CNN
-	1    9550 4050
-	1    0    0    -1
-$EndComp
-Text GLabel 10000 4050 2    60   Input ~ 0
-GND
-Wire Wire Line
-	10000 4050 9850 4050
+P 9550 4200
+F 0 "SW1" H 9700 4310 50  0000 C CNN
+F 1 "SW_PUSH" H 9550 4120 50  0000 C CNN
+F 2 "" H 9550 4200 60  0001 C CNN
+F 3 "" H 9550 4200 60  0000 C CNN
+	1    9550 4200
+	1    0    0    -1
+$EndComp
+Text GLabel 10000 4200 2    60   Input ~ 0
+GND
+Wire Wire Line
+	10000 4200 9850 4200
 $Comp
 L R R1
 U 1 1 55F95FFC
-P 9050 4350
-F 0 "R1" V 9130 4350 50  0000 C CNN
-F 1 "10K" V 9050 4350 50  0000 C CNN
-F 2 "" V 8980 4350 30  0000 C CNN
-F 3 "" H 9050 4350 30  0000 C CNN
-	1    9050 4350
-	1    0    0    -1
-$EndComp
-Wire Wire Line
-	9050 4200 9050 4050
-Connection ~ 9050 4050
-Text GLabel 9050 4650 3    60   Input ~ 0
-VCC
-Wire Wire Line
-	9050 4650 9050 4500
-Text GLabel 8900 4050 0    60   Input ~ 0
+P 9050 4500
+F 0 "R1" V 9130 4500 50  0000 C CNN
+F 1 "10K" V 9050 4500 50  0000 C CNN
+F 2 "Resistors_ThroughHole:Resistor_Horizontal_RM10mm" V 8980 4500 30  0001 C CNN
+F 3 "" H 9050 4500 30  0000 C CNN
+	1    9050 4500
+	1    0    0    -1
+$EndComp
+Wire Wire Line
+	9050 4350 9050 4200
+Connection ~ 9050 4200
+Text GLabel 9050 4800 3    60   Input ~ 0
+VCC
+Wire Wire Line
+	9050 4800 9050 4650
+Text GLabel 8900 4200 0    60   Input ~ 0
 RST
 Wire Wire Line
 	9000 2500 8850 2500
 Wire Wire Line
-	8900 4050 9250 4050
-Wire Notes Line
-	10550 4950 7900 4950
-Wire Notes Line
-	7900 4950 7900 3850
-Wire Notes Line
-	7900 3850 10550 3850
-Wire Notes Line
-	10550 3850 10550 4950
-Text Notes 9850 4900 0    60   ~ 0
+	8900 4200 9250 4200
+Wire Notes Line
+	10550 5100 7900 5100
+Wire Notes Line
+	7900 5100 7900 4000
+Wire Notes Line
+	7900 4000 10550 4000
+Wire Notes Line
+	10550 4000 10550 5100
+Text Notes 9850 5050 0    60   ~ 0
 RESET CIRCUIT
 Wire Wire Line
@@
 F 0 "P1" H 1500 1100 50  0000 C CNN
 F 1 "SERVO_HEADER" V 1600 900 50  0000 C CNN
-F 2 "" H 1500 900 60  0000 C CNN
+F 2 "Pin_Headers:Pin_Header_Angled_1x03" H 1500 900 60  0001 C CNN
 F 3 "" H 1500 900 60  0000 C CNN
 	1    1500 900
@@
 F 0 "P5" H 2250 1100 50  0000 C CNN
 F 1 "SERVO_HEADER" V 2350 900 50  0000 C CNN
-F 2 "" H 2250 900 60  0000 C CNN
+F 2 "Pin_Headers:Pin_Header_Angled_1x03" H 2250 900 60  0001 C CNN
 F 3 "" H 2250 900 60  0000 C CNN
 	1    2250 900
@@
 F 0 "P9" H 3000 1100 50  0000 C CNN
 F 1 "SERVO_HEADER" V 3100 900 50  0000 C CNN
-F 2 "" H 3000 900 60  0000 C CNN
+F 2 "Pin_Headers:Pin_Header_Angled_1x03" H 3000 900 60  0001 C CNN
 F 3 "" H 3000 900 60  0000 C CNN
 	1    3000 900
@@
 F 0 "P2" H 1500 1950 50  0000 C CNN
 F 1 "SERVO_HEADER" V 1600 1750 50  0000 C CNN
-F 2 "" H 1500 1750 60  0000 C CNN
+F 2 "Pin_Headers:Pin_Header_Angled_1x03" H 1500 1750 60  0001 C CNN
 F 3 "" H 1500 1750 60  0000 C CNN
 	1    1500 1750
@@
 F 0 "P6" H 2250 1950 50  0000 C CNN
 F 1 "SERVO_HEADER" V 2350 1750 50  0000 C CNN
-F 2 "" H 2250 1750 60  0000 C CNN
+F 2 "Pin_Headers:Pin_Header_Angled_1x03" H 2250 1750 60  0001 C CNN
 F 3 "" H 2250 1750 60  0000 C CNN
 	1    2250 1750
@@
 F 0 "P10" H 3000 1950 50  0000 C CNN
 F 1 "SERVO_HEADER" V 3100 1750 50  0000 C CNN
-F 2 "" H 3000 1750 60  0000 C CNN
+F 2 "Pin_Headers:Pin_Header_Angled_1x03" H 3000 1750 60  0001 C CNN
 F 3 "" H 3000 1750 60  0000 C CNN
 	1    3000 1750
@@
 F 0 "P3" H 1500 2800 50  0000 C CNN
 F 1 "SERVO_HEADER" V 1600 2600 50  0000 C CNN
-F 2 "" H 1500 2600 60  0000 C CNN
+F 2 "Pin_Headers:Pin_Header_Angled_1x03" H 1500 2600 60  0001 C CNN
 F 3 "" H 1500 2600 60  0000 C CNN
 	1    1500 2600
@@
 F 0 "P7" H 2250 2800 50  0000 C CNN
 F 1 "SERVO_HEADER" V 2350 2600 50  0000 C CNN
-F 2 "" H 2250 2600 60  0000 C CNN
+F 2 "Pin_Headers:Pin_Header_Angled_1x03" H 2250 2600 60  0001 C CNN
 F 3 "" H 2250 2600 60  0000 C CNN
 	1    2250 2600
@@
 F 0 "P11" H 3000 2800 50  0000 C CNN
 F 1 "SERVO_HEADER" V 3100 2600 50  0000 C CNN
-F 2 "" H 3000 2600 60  0000 C CNN
+F 2 "Pin_Headers:Pin_Header_Angled_1x03" H 3000 2600 60  0001 C CNN
 F 3 "" H 3000 2600 60  0000 C CNN
 	1    3000 2600
@@
 F 0 "P4" H 1500 3650 50  0000 C CNN
 F 1 "SERVO_HEADER" V 1600 3450 50  0000 C CNN
-F 2 "" H 1500 3450 60  0000 C CNN
+F 2 "Pin_Headers:Pin_Header_Angled_1x03" H 1500 3450 60  0001 C CNN
 F 3 "" H 1500 3450 60  0000 C CNN
 	1    1500 3450
@@
 F 0 "P8" H 2250 3650 50  0000 C CNN
 F 1 "SERVO_HEADER" V 2350 3450 50  0000 C CNN
-F 2 "" H 2250 3450 60  0000 C CNN
+F 2 "Pin_Headers:Pin_Header_Angled_1x03" H 2250 3450 60  0001 C CNN
 F 3 "" H 2250 3450 60  0000 C CNN
 	1    2250 3450
@@
 F 0 "P12" H 3000 3650 50  0000 C CNN
 F 1 "SERVO_HEADER" V 3100 3450 50  0000 C CNN
-F 2 "" H 3000 3450 60  0000 C CNN
+F 2 "Pin_Headers:Pin_Header_Angled_1x03" H 3000 3450 60  0001 C CNN
 F 3 "" H 3000 3450 60  0000 C CNN
 	1    3000 3450
@@
 F 0 "Y1" H 9150 1850 50  0000 C CNN
 F 1 "16MHz" V 9150 1550 50  0000 C CNN
-F 2 "" H 9150 1750 60  0000 C CNN
+F 2 "Crystals:Crystal_HC49-U_Vertical" H 9150 1750 60  0001 C CNN
 F 3 "" H 9150 1750 60  0000 C CNN
 	1    9150 1750
@@
 F 0 "C1" H 9725 1750 50  0000 L CNN
 F 1 "22pF" H 9500 1550 50  0000 L CNN
-F 2 "" H 9738 1500 30  0000 C CNN
+F 2 "Capacitors_ThroughHole:C_Disc_D3_P2.5" H 9738 1500 30  0001 C CNN
 F 3 "" H 9700 1650 60  0000 C CNN
 	1    9700 1650
@@
 F 0 "C2" H 9725 1950 50  0000 L CNN
 F 1 "22pF" H 9725 1750 50  0000 L CNN
-F 2 "" H 9738 1700 30  0000 C CNN
+F 2 "Capacitors_ThroughHole:C_Disc_D3_P2.5" H 9738 1700 30  0001 C CNN
 F 3 "" H 9700 1850 60  0000 C CNN
 	1    9700 1850
@@
 Connection ~ 10000 1750
 $Comp
-L BARREL_JACK CON?
+L BARREL_JACK CON2
 U 1 1 55F99D4A
 P 1800 5250
-F 0 "CON?" H 1800 5500 60  0000 C CNN
+F 0 "CON2" H 1800 5500 60  0000 C CNN
 F 1 "BARREL_JACK" H 1800 5050 60  0000 C CNN
-F 2 "" H 1800 5250 60  0000 C CNN
+F 2 "library:BARREL_JACK" H 1800 5250 60  0001 C CNN
 F 3 "" H 1800 5250 60  0000 C CNN
 	1    1800 5250
@@
 $EndComp
 $Comp
-L LM7805 U?
+L LM7805 U1
 U 1 1 55F99DFD
 P 3050 5200
-F 0 "U?" H 3200 5004 60  0000 C CNN
+F 0 "U1" H 3200 5004 60  0000 C CNN
 F 1 "LM7805" H 3050 5400 60  0000 C CNN
-F 2 "" H 3050 5200 60  0000 C CNN
+F 2 "library:LM7805" H 3050 5200 60  0001 C CNN
 F 3 "" H 3050 5200 60  0000 C CNN
 	1    3050 5200
@@
 VCC
 $Comp
-L C C?
+L C C3
 U 1 1 55F9A6BA
 P 2500 5450
-F 0 "C?" H 2525 5550 50  0000 L CNN
+F 0 "C3" H 2525 5550 50  0000 L CNN
 F 1 "100nF" H 2250 5350 50  0000 L CNN
-F 2 "" H 2538 5300 30  0000 C CNN
+F 2 "Capacitors_ThroughHole:C_Radial_D10_L13_P5" H 2538 5300 30  0001 C CNN
 F 3 "" H 2500 5450 60  0000 C CNN
 	1    2500 5450
@@
 	2500 5150 2500 5300
 $Comp
-L C C?
+L C C4
 U 1 1 55F9AD53
 P 3550 5450
-F 0 "C?" H 3575 5550 50  0000 L CNN
+F 0 "C4" H 3575 5550 50  0000 L CNN
 F 1 "10nF" H 3575 5350 50  0000 L CNN
-F 2 "" H 3588 5300 30  0000 C CNN
+F 2 "Capacitors_ThroughHole:C_Radial_D5_L6_P2.5" H 3588 5300 30  0001 C CNN
 F 3 "" H 3550 5450 60  0000 C CNN
 	1    3550 5450
@@
 	3550 5650 3550 5600
 $Comp
-L CONN_01X06 P?
+L CONN_01X06 P13
 U 1 1 55F9C036
-P 10500 2700
-F 0 "P?" H 10500 3050 50  0000 C CNN
-F 1 "Bluetooth_header" V 10600 2700 50  0000 C CNN
-F 2 "" H 10500 2700 60  0000 C CNN
-F 3 "" H 10500 2700 60  0000 C CNN
-	1    10500 2700
-	1    0    0    -1
-$EndComp
-Wire Wire Line
-	9950 2850 10300 2850
-Wire Wire Line
-	10200 2750 10300 2750
-Text GLabel 9950 2650 0    60   Input ~ 0
+P 7600 5650
+F 0 "P13" H 7600 6000 50  0000 C CNN
+F 1 "Bluetooth_header" V 7700 5650 50  0000 C CNN
+F 2 "Pin_Headers:Pin_Header_Angled_1x06" H 7600 5650 60  0001 C CNN
+F 3 "" H 7600 5650 60  0000 C CNN
+	1    7600 5650
+	1    0    0    -1
+$EndComp
+Wire Wire Line
+	7050 5800 7400 5800
+Wire Wire Line
+	7300 5700 7400 5700
+Text GLabel 7050 5600 0    60   Input ~ 0
 BTX
 Wire Wire Line
-	9950 2650 10300 2650
-Text GLabel 10200 2550 0    60   Input ~ 0
+	7050 5600 7400 5600
+Text GLabel 6700 5400 0    60   Input ~ 0
 BRX
-Wire Wire Line
-	10200 2550 10300 2550
 Text GLabel 9250 2750 2    60   Input ~ 0
 BRX
@@
 Wire Wire Line
 	9000 2650 8850 2650
+$Comp
+L R R2
+U 1 1 55F9D523
+P 6950 5400
+F 0 "R2" V 7030 5400 50  0000 C CNN
+F 1 "330" V 6950 5400 50  0000 C CNN
+F 2 "Resistors_ThroughHole:Resistor_Horizontal_RM10mm" V 6880 5400 30  0001 C CNN
+F 3 "" H 6950 5400 30  0000 C CNN
+	1    6950 5400
+	0    -1   -1   0
+$EndComp
+Wire Wire Line
+	6800 5400 6700 5400
+Wire Wire Line
+	7100 5400 7150 5400
+Wire Wire Line
+	7150 5300 7150 5500
+Wire Wire Line
+	7150 5500 7400 5500
+Connection ~ 7150 5400
+$Comp
+L R R3
+U 1 1 55F9DB47
+P 7150 5150
+F 0 "R3" V 7230 5150 50  0000 C CNN
+F 1 "660" V 7150 5150 50  0000 C CNN
+F 2 "Resistors_ThroughHole:Resistor_Horizontal_RM10mm" V 7080 5150 30  0001 C CNN
+F 3 "" H 7150 5150 30  0000 C CNN
+	1    7150 5150
+	-1   0    0    1
+$EndComp
+Text GLabel 7150 4950 1    60   Input ~ 0
+GND
+Wire Wire Line
+	7150 4950 7150 5000
+Wire Notes Line
+	7850 6250 7850 4650
+Wire Notes Line
+	7850 4650 6250 4650
+Wire Notes Line
+	6250 4650 6250 6250
+Wire Notes Line
+	6250 6250 7850 6250
+Text Notes 6800 6200 0    60   ~ 0
+BLUETOOTH CIRCUIT
+Wire Notes Line
+	4150 6050 1050 6050
+Wire Notes Line
+	1050 6050 1050 4800
+Wire Notes Line
+	1050 4800 4150 4800
+Wire Notes Line
+	4150 4800 4150 6050
+Text Notes 3400 6000 0    60   ~ 0
+POWER CIRCUIT
 $EndSCHEMATC
